Commit message: Fixing G1 Robot error in not appearing in Gazebo

File: sam_simulation/urdf/g1_sensors.urdf.xacro (robot description, xacro)
@@ -1,29 +1,159 @@
 <?xml version="1.0"?>
 <robot name="g1_humanoid_sim" xmlns:xacro="http://ros.org/wiki/xacro">
-  <!-- Base Link (The Robot's Body) -->
+  <!-- ================================================================
+       G1 Humanoid — Simplified Visual Model for Simulation
+       Body is built from primitive shapes (box, cylinder, sphere).
+       All sensor plugins are attached at anatomically correct positions.
+       ================================================================ -->
+  <!-- Torso (main body) -->
   <link name="base_link">
     <visual>
-      <geometry><cylinder radius="0.2" length="1.0"/></geometry>
-      <material name="gray"><color rgba="0.5 0.5 0.5 1"/></material>
+      <geometry><box size="0.35 0.25 0.5"/></geometry>
+      <material name="dark_gray"><color rgba="0.2 0.2 0.2 1"/></material>
     </visual>
-    <collision><geometry><cylinder radius="0.2" length="1.0"/></geometry></collision>
-    <inertial><mass value="10.0"/><inertia ixx="0.1" ixy="0" ixz="0" iyy="0.1" iyz="0" izz="0.1"/></inertial>
+    <collision><geometry><box size="0.35 0.25 0.5"/></geometry></collision>
+    <inertial>
+      <mass value="30.0"/>
+      <inertia ixx="0.5" ixy="0" ixz="0" iyy="0.5" iyz="0" izz="0.3"/>
+    </inertial>
   </link>
-  <!-- RGB-D Camera Link (Head) -->
+  <!-- Head -->
+  <link name="head_link">
+    <visual>
+      <geometry><sphere radius="0.12"/></geometry>
+      <material name="light_gray"><color rgba="0.7 0.7 0.7 1"/></material>
+    </visual>
+    <collision><geometry><sphere radius="0.12"/></geometry></collision>
+    <inertial><mass value="2.0"/><inertia ixx="0.01" ixy="0" ixz="0" iyy="0.01" iyz="0" izz="0.01"/></inertial>
+  </link>
+  <joint name="neck_joint" type="fixed">
+    <parent link="base_link"/><child link="head_link"/>
+    <origin xyz="0 0 0.35" rpy="0 0 0"/>
+  </joint>
+  <!-- Left Upper Arm -->
+  <link name="left_upper_arm">
+    <visual>
+      <geometry><cylinder radius="0.05" length="0.28"/></geometry>
+      <material name="dark_gray"><color rgba="0.2 0.2 0.2 1"/></material>
+    </visual>
+    <collision><geometry><cylinder radius="0.05" length="0.28"/></cylinder></geometry></collision>
+    <inertial><mass value="2.0"/><inertia ixx="0.01" ixy="0" ixz="0" iyy="0.01" iyz="0" izz="0.01"/></inertial>
+  </link>
+  <joint name="left_shoulder_joint" type="fixed">
+    <parent link="base_link"/><child link="left_upper_arm"/>
+    <origin xyz="0 0.2 0.15" rpy="0 0 0"/>
+  </joint>
+  <!-- Right Upper Arm -->
+  <link name="right_upper_arm">
+    <visual>
+      <geometry><cylinder radius="0.05" length="0.28"/></geometry>
+      <material name="dark_gray"><color rgba="0.2 0.2 0.2 1"/></material>
+    </visual>
+    <collision><geometry><cylinder radius="0.05" length="0.28"/></cylinder></geometry></collision>
+    <inertial><mass value="2.0"/><inertia ixx="0.01" ixy="0" ixz="0" iyy="0.01" iyz="0" izz="0.01"/></inertial>
+  </link>
+  <joint name="right_shoulder_joint" type="fixed">
+    <parent link="base_link"/><child link="right_upper_arm"/>
+    <origin xyz="0 -0.2 0.15" rpy="0 0 0"/>
+  </joint>
+  <!-- Left Lower Arm -->
+  <link name="left_lower_arm">
+    <visual>
+      <geometry><cylinder radius="0.04" length="0.26"/></geometry>
+      <material name="light_gray"><color rgba="0.7 0.7 0.7 1"/></material>
+    </visual>
+    <collision><geometry><cylinder radius="0.04" length="0.26"/></cylinder></geometry></collision>
+    <inertial><mass value="1.0"/><inertia ixx="0.005" ixy="0" ixz="0" iyy="0.005" iyz="0" izz="0.005"/></inertial>
+  </link>
+  <joint name="left_elbow_joint" type="fixed">
+    <parent link="left_upper_arm"/><child link="left_lower_arm"/>
+    <origin xyz="0 0 -0.27" rpy="0 0 0"/>
+  </joint>
+  <!-- Right Lower Arm -->
+  <link name="right_lower_arm">
+    <visual>
+      <geometry><cylinder radius="0.04" length="0.26"/></geometry>
+      <material name="light_gray"><color rgba="0.7 0.7 0.7 1"/></material>
+    </visual>
+    <collision><geometry><cylinder radius="0.04" length="0.26"/></cylinder></geometry></collision>
+    <inertial><mass value="1.0"/><inertia ixx="0.005" ixy="0" ixz="0" iyy="0.005" iyz="0" izz="0.005"/></inertial>
+  </link>
+  <joint name="right_elbow_joint" type="fixed">
+    <parent link="right_upper_arm"/><child link="right_lower_arm"/>
+    <origin xyz="0 0 -0.27" rpy="0 0 0"/>
+  </joint>
+  <!-- Left Thigh -->
+  <link name="left_thigh">
+    <visual>
+      <geometry><cylinder radius="0.07" length="0.35"/></geometry>
+      <material name="dark_gray"><color rgba="0.2 0.2 0.2 1"/></material>
+    </visual>
+    <collision><geometry><cylinder radius="0.07" length="0.35"/></cylinder></geometry></collision>
+    <inertial><mass value="5.0"/><inertia ixx="0.05" ixy="0" ixz="0" iyy="0.05" iyz="0" izz="0.02"/></inertial>
+  </link>
+  <joint name="left_hip_joint" type="fixed">
+    <parent link="base_link"/><child link="left_thigh"/>
+    <origin xyz="0 0.1 -0.42" rpy="0 0 0"/>
+  </joint>
+  <!-- Right Thigh -->
+  <link name="right_thigh">
+    <visual>
+      <geometry><cylinder radius="0.07" length="0.35"/></geometry>
+      <material name="dark_gray"><color rgba="0.2 0.2 0.2 1"/></material>
+    </visual>
+    <collision><geometry><cylinder radius="0.07" length="0.35"/></cylinder></geometry></collision>
+    <inertial><mass value="5.0"/><inertia ixx="0.05" ixy="0" ixz="0" iyy="0.05" iyz="0" izz="0.02"/></inertial>
+  </link>
+  <joint name="right_hip_joint" type="fixed">
+    <parent link="base_link"/><child link="right_thigh"/>
+    <origin xyz="0 -0.1 -0.42" rpy="0 0 0"/>
+  </joint>
+  <!-- Left Shin -->
+  <link name="left_shin">
+    <visual>
+      <geometry><cylinder radius="0.055" length="0.33"/></geometry>
+      <material name="light_gray"><color rgba="0.7 0.7 0.7 1"/></material>
+    </visual>
+    <collision><geometry><cylinder radius="0.055" length="0.33"/></cylinder></geometry></collision>
+    <inertial><mass value="3.0"/><inertia ixx="0.03" ixy="0" ixz="0" iyy="0.03" iyz="0" izz="0.01"/></inertial>
+  </link>
+  <joint name="left_knee_joint" type="fixed">
+    <parent link="left_thigh"/><child link="left_shin"/>
+    <origin xyz="0 0 -0.34" rpy="0 0 0"/>
+  </joint>
+  <!-- Right Shin -->
+  <link name="right_shin">
+    <visual>
+      <geometry><cylinder radius="0.055" length="0.33"/></geometry>
+      <material name="light_gray"><color rgba="0.7 0.7 0.7 1"/></material>
+    </visual>
+    <collision><geometry><cylinder radius="0.055" length="0.33"/></cylinder></geometry></collision>
+    <inertial><mass value="3.0"/><inertia ixx="0.03" ixy="0" ixz="0" iyy="0.03" iyz="0" izz="0.01"/></inertial>
+  </link>
+  <joint name="right_knee_joint" type="fixed">
+    <parent link="right_thigh"/><child link="right_shin"/>
+    <origin xyz="0 0 -0.34" rpy="0 0 0"/>
+  </joint>
+  <!-- ================================================================
+       SENSOR LINKS — Attached at anatomically correct positions
+       ================================================================ -->
+  <!-- RGB-D Camera — mounted at head level, facing forward -->
   <link name="camera_link"/>
   <joint name="camera_joint" type="fixed">
-    <parent link="base_link"/>
+    <parent link="head_link"/>
     <child link="camera_link"/>
-    <origin xyz="0.1 0 0.5" rpy="0 0 0"/>
+    <origin xyz="0.12 0 0" rpy="0 0 0"/>
   </joint>
-  <!-- LiDAR Link (Torso) -->
+  <!-- LiDAR — mounted on top of the torso -->
   <link name="lidar_link"/>
   <joint name="lidar_joint" type="fixed">
     <parent link="base_link"/>
     <child link="lidar_link"/>
-    <origin xyz="0 0 0.2" rpy="0 0 0"/>
+    <origin xyz="0 0 0.28" rpy="0 0 0"/>
   </joint>
-  <!-- ================= GAZEBO PLUGINS ================= -->
-  <!-- RGB-D Camera Plugin -->
+  <!-- ================================================================
+       GAZEBO SENSOR PLUGINS
+       ================================================================ -->
+  <!-- RGB-D Depth Camera Plugin -->
   <gazebo reference="camera_link">
     <sensor name="camera" type="depth">
@@ -41,5 +171,5 @@
     </sensor>
   </gazebo>
-  <!-- 2D LiDAR Plugin (Cartographer uses this) -->
+  <!-- 2D LiDAR Plugin -->
   <gazebo reference="lidar_link">
     <sensor name="lidar" type="ray">
@@ -48,5 +178,10 @@
       <update_rate>10.0</update_rate>
       <ray>
-        <scan><horizontal><samples>360</samples><resolution>1</resolution><min_angle>-3.14</min_angle><max_angle>3.14</max_angle></horizontal></scan>
+        <scan>
+          <horizontal>
+            <samples>360</samples><resolution>1</resolution>
+            <min_angle>-3.14159</min_angle><max_angle>3.14159</max_angle>
+          </horizontal>
+        </scan>
         <range><min>0.12</min><max>10.0</max></range>
       </ray>
