Commit message: Fixing Algorithms integrations inside gazebo environment && Adding DeepLabV3 algorithm

File: g1_description/g1_23dof.urdf (robot description, URDF)
Before this commit: robot g1_23dof, 33 links, 32 joints
Links:
- added link camera_depth_optical_frame
- link d435_link: mass None -> 0.001; geometry visual box size=0.01 0.03 0.01
Joints:
- added joint camera_optical_joint: type fixed, parent d435_link, child camera_depth_optical_frame, origin xyz=0 0 0 rpy=-1.5707963 0 -1.5707963
